File: Power options/Reset button/sc_reset/sc_reset.kicad_pcb (KiCad board)
At the start: 2 copper layers, 13.1 x 27.7 mm, 4 parts, among them J1 Conn_02x05_Odd_Even

Commit message: Reset pcb
Parts:
- removed H2: MountingHole, MountingHole:MountingHole_3.2mm_M3
Other:
- board size 13.1 x 27.7 mm -> 13.1 x 21.8 mm
Changed lines of the file:
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@@
   (general
     (thickness 1.6)
-    (drawings 12)
+    (drawings 10)
     (tracks 14)
     (zones 0)
-    (modules 4)
+    (modules 3)
     (nets 3)
   )
@@
     (39 F.Mask user)
     (40 Dwgs.User user)
-    (41 Cmts.User user)
+    (41 Cmts.User user hide)
     (42 Eco1.User user)
     (43 Eco2.User user)
@@
     (46 B.CrtYd user hide)
     (47 F.CrtYd user hide)
-    (48 B.Fab user)
+    (48 B.Fab user hide)
     (49 F.Fab user hide)
   )
@@
     (uvia_dia 0.3)
     (uvia_drill 0.1)
-    (add_net "Net-(J1-Pad1)")
     (add_net "Net-(J1-Pad10)")
-    (add_net "Net-(J1-Pad2)")
-    (add_net "Net-(J1-Pad3)")
-    (add_net "Net-(J1-Pad4)")
-    (add_net "Net-(J1-Pad5)")
-    (add_net "Net-(J1-Pad6)")
-    (add_net "Net-(J1-Pad7)")
-    (add_net "Net-(J1-Pad8)")
     (add_net "Net-(J1-Pad9)")
-  )
-  (module MountingHole:MountingHole_3.2mm_M3 (layer F.Cu)
-    (at 151.8 117.51)
-    (descr "Mounting Hole 3.2mm, no annular, M3")
-    (tags "mounting hole 3.2mm no annular m3")
-    (attr virtual)
-    (fp_text reference H2 (at 0 -4.2) (layer F.SilkS)
-      (effects (font (size 1 1) (thickness 0.15)))
-    )
-    (fp_text value MountingHole (at 0 4.2) (layer F.Fab)
-      (effects (font (size 1 1) (thickness 0.15)))
-    )
-    (fp_text user %R (at 0.3 0) (layer F.Fab)
-      (effects (font (size 1 1) (thickness 0.15)))
-    )
-    (fp_circle (center 0 0) (end 3.2 0) (layer Cmts.User) (width 0.15))
-    (fp_circle (center 0 0) (end 3.45 0) (layer F.CrtYd) (width 0.05))
-    (pad 1 np_thru_hole circle (at 0 0) (size 3.2 3.2) (drill 3.2) (layers *.Cu *.Mask))
   )
   (module fab:TACTILE-SWITCH-12mm-5mmH (layer F.Cu)
@@
     )
   )
-  (gr_arc (start 156.787875 100.799999) (end 158.05 99.84) (angle 36.9) (layer Edge.Cuts) (width 0.05))
-  (gr_arc (start 151.8 96.24) (end 154.475 94.44) (angle -112.1) (layer Edge.Cuts) (width 0.05))
-  (gr_line (start 149.125849 94.43874) (end 145.550849 99.83874) (layer Edge.Cuts) (width 0.05))
-  (gr_line (start 154.475 94.44) (end 158.05 99.84) (layer Edge.Cuts) (width 0.05))
-  (gr_arc (start 146.812974 100.798739) (end 145.550849 99.83874) (angle -36.9) (layer Edge.Cuts) (width 0.05))
-  (gr_line (start 149.125 119.3) (end 145.55 113.9) (layer Edge.Cuts) (width 0.05))
-  (gr_line (start 145.226421 112.949891) (end 145.227269 100.788848) (layer Edge.Cuts) (width 0.05))
-  (gr_arc (start 146.812126 112.94) (end 145.550001 113.899999) (angle 36.9) (layer Edge.Cuts) (width 0.05))
-  (gr_arc (start 156.787874 112.94) (end 158.049999 113.899999) (angle -36.9) (layer Edge.Cuts) (width 0.05))
-  (gr_arc (start 151.8 117.5) (end 149.125 119.3) (angle -112.1) (layer Edge.Cuts) (width 0.05))
-  (gr_line (start 154.475 119.3) (end 158.05 113.9) (layer Edge.Cuts) (width 0.05))
-  (gr_line (start 158.373579 112.949891) (end 158.37358 100.790108) (layer Edge.Cuts) (width 0.05))
+  (gr_arc (start 147.046421 112.949891) (end 147.046421 114.769891) (angle 90) (layer Edge.Cuts) (width 0.2))
+  (gr_arc (start 156.553579 112.949891) (end 156.553579 114.769891) (angle -90) (layer Edge.Cuts) (width 0.2))
+  (gr_line (start 147.046421 114.769891) (end 156.553579 114.769891) (layer Edge.Cuts) (width 0.2))
+  (gr_arc (start 156.787875 100.799999) (end 158.05 99.84) (angle 36.9) (layer Edge.Cuts) (width 0.2))
+  (gr_arc (start 151.8 96.24) (end 154.475 94.44) (angle -112.1) (layer Edge.Cuts) (width 0.2))
+  (gr_line (start 149.125849 94.43874) (end 145.550849 99.83874) (layer Edge.Cuts) (width 0.2))
+  (gr_line (start 154.475 94.44) (end 158.05 99.84) (layer Edge.Cuts) (width 0.2))
+  (gr_arc (start 146.812974 100.798739) (end 145.550849 99.83874) (angle -36.9) (layer Edge.Cuts) (width 0.2))
+  (gr_line (start 145.226421 112.949891) (end 145.227269 100.788848) (layer Edge.Cuts) (width 0.2))
+  (gr_line (start 158.373579 112.949891) (end 158.37358 100.790108) (layer Edge.Cuts) (width 0.2))
   (segment (start 153.7 100.325) (end 154.25 100.875) (width 0.5) (layer F.Cu) (net 1))
   (segment (start 154.25 110) (end 153.64 109.39) (width 0.5) (layer F.Cu) (net 1))
