File: Power options/Power hub/power-routing/power-routing.sch (KiCad schematic (older format))
At the start: 13 parts, among them J1 Input_Bulgin, J2 Screw_Terminal_01x02, J3 Screw_Terminal_01x02, J4 Screw_Terminal_01x02, J6 USB_A, M1 RED, U1 fablab, U2 smartcitizen

Commit message: Update power hub
Parts:
- M1: LCSC (none) -> C93133
- R1: value 220Ω -> 1000Ω; LCSC (none) -> C4410
Changed lines of the file:
@@
 F 2 "LED_SMD:LED_1206_3216Metric_Pad1.42x1.75mm_HandSolder" H 5580 3050 20  0001 C CNN
 F 3 "" H 5550 2900 50  0001 C CNN
+F 4 "C93133" H 5550 2900 50  0001 C CNN "LCSC"
 	1    5550 2900
 	1    0    0    -1
@@
 P 5900 2850
 F 0 "R1" V 5858 2918 45  0000 L CNN
-F 1 "220Ω" V 5942 2918 45  0000 L CNN
+F 1 "1000Ω" V 5942 2918 45  0000 L CNN
 F 2 "fab-R1206FAB" H 5930 3000 20  0001 C CNN
 F 3 "" H 5900 2850 50  0001 C CNN
+F 4 "C4410" V 5900 2850 50  0001 C CNN "LCSC"
 	1    5900 2850
 	0    1    1    0
